File: motordriver2.kicad_sch (KiCad schematic)
At the start: 37 parts, among them M1 Motor_DC, Q1 TPHR9003NL, Q2 TPHR9003NL, Q3 TPHR9003NL, Q4 TPHR9003NL, U1 PLM2105DR, U2 PLM2105DR, U4 MC78M05_TO252, U5 AMS1117-3.3

Commit message: add power source
Parts:
- removed D6: SS34, Diode_SMD:D_MELF, symbol Device:D
- removed U4: MC78M05_TO252, Package_TO_SOT_SMD:TO-252-2, symbol Regulator_Linear:MC78M05_TO252
- added C10: CL31B105KBHNNNE, symbol Device:C
- added C11: CL21A226MAQNNNE, symbol Device:C
- added C12, C13, C14, C23: CL05B104KO5NNNC, Capacitor_SMD:C_0402_1005Metric, symbol Device:C
- added C15: CL05B103KB5NNNC, Capacitor_SMD:C_0402_1005Metric, symbol Device:C
- added C16: CL10A105KB8NNNC, Capacitor_SMD:C_0603_1608Metric, symbol Device:C
- added C17, C18, C21, C22: 0402CG150J500NT, Capacitor_SMD:C_0402_1005Metric, symbol Device:C
- added C19, C20: CL05C100JB5NNNC, symbol Device:C
- added C24: CL10A475KO8NNNC, Capacitor_SMD:C_0603_1608Metric, symbol Device:C
- added D10, D11, D12, D13, D14, D16, D17, D18, D19, D8, D9: ESD3Z5.0C, Diode_SMD:D_SOD-323, symbol Device:D_TVS
- added D15, D20, D6: ES0402V014BT, Diode_SMD:D_0402_1005Metric, symbol Device:D_TVS
- added D21, D22, D7: SS34, Diode_SMD:D_MELF, symbol Device:D
- added J1, J3: DE9_Receptacle_MountingHoles, symbol Connector:DE9_Receptacle_MountingHoles
- added J2: Conn_01x06_Pin, Connector_PinSocket_2.54mm:PinSocket_1x06_P2.54mm_Vertical, symbol Connector:Conn_01x06_Pin
- added J4: Conn_01x03_Pin, Connector_PinSocket_2.54mm:PinSocket_1x03_P2.54mm_Vertical, symbol Connector:Conn_01x03_Pin
- added J5: Conn_01x02_Pin, Connector_AMASS:AMASS_XT60IPW-M_1x03_P7.20mm_Horizontal, symbol Connector:Conn_01x02_Pin
- added JP1: Jumper_2_Open, Jumper:SolderJumper-2_P1.3mm_Open_Pad1.0x1.5mm, symbol Jumper:Jumper_2_Open
- added R14, R16, R17, R18, R19, R23, R24, R25, R27: 0805W8F100JT5E, Resistor_SMD:R_0805_2012Metric, symbol Device:R
- added R15, R20, R26, R28: 0402WGF1002TCE, Resistor_SMD:R_0402_1005Metric, symbol Device:R
- added R21, R22, R29, R30: R, symbol Device:R
- added R31, R32: 0805W8F3301T5E, Resistor_SMD:R_0805_2012Metric, symbol Device:R
- added RV1, RV2: SDV1608H260C050YPTF, Resistor_SMD:R_0603_1608Metric, symbol Device:Varistor
- added SW1, SW2, SW3: SW_Push, symbol Switch:SW_Push
- added TP1, TP2, TP3, TP4: TestPoint, TestPoint:TestPoint_Loop_D1.80mm_Drill1.0mm_Beaded, symbol Connector:TestPoint
- added U3: STM32F302C8Tx, Package_QFP:LQFP-48_7x7mm_P0.5mm, symbol MCU_ST_STM32F3:STM32F302C8Tx
- added U4: AMS1117-3.3, Package_TO_SOT_SMD:SOT-223-3_TabPin2, symbol Regulator_Linear:AMS1117-3.3
- added U6: SN65HVD234, Package_SO:SOIC-8_3.9x4.9mm_P1.27mm, symbol Interface_CAN_LIN:SN65HVD234
- added U7: 24LC256, symbol Memory_EEPROM:24LC256
- added Y1: X322516MLB4SI, symbol Device:Crystal
- added Y2: Q13FC1350000400, symbol Device:Crystal
- C6: value CL31B105KBHNNNE -> CL05B104KO5NNNC; footprint (none) -> Capacitor_SMD:C_0402_1005Metric; LCSC C1848 -> C1525
- C7: value CL31B105KBHNNNE -> CL10A475KO8NNNC; footprint (none) -> Capacitor_SMD:C_0603_1608Metric; LCSC C1848 -> C19666
- D5: value SS34 -> ESD9X3.3ST5G; footprint Diode_SMD:D_MELF -> Diode_SMD:D_SOD-923; LCSC C8678 -> C130456
- M1: footprint (none) -> Connector_AMASS:AMASS_XT60PW-F_1x02_P7.20mm_Horizontal
Connections:
- net +3.3V: now also C6.1, C7.1, C12.1, C13.1, C14.1, C23.1, C24.1, D13.2 (A2), D21.2 (A), D7.2 (A), J2.1 (Pin_1), R15.1, R20.1, R21.1, R26.1, R28.1, R31.1, R32.1, U3.1 (VBAT), U3.24 (VDD), U3.36 (VDD), U3.48 (VDD), U6.3 (VCC), U7.8 (VCC); no longer D5.1 (K)
- net GATEHA: now also U3.29 (PA8)
- net GATEHB: now also U3.31 (PA10)
- net GATELA: now also U3.2 (PC13)
- net GATELB: now also U3.28 (PB15)
- net GND: now also D5.2 (A), C10.2, C11.2, C12.2, C13.2, C14.2, C15.2, C16.2, C17.1, C18.1, C19.1, C20.1, C21.1, C22.2, C23.2, C24.2, D10.1 (A1), D11.1 (A1), D12.1 (A1), D13.1 (A1), D14.1 (A1), D15.1 (A1), D16.1 (A1), D17.1 (A1), D18.1 (A1), D19.1 (A1), D20.1 (A1), D6.1 (A1), D8.2 (A2), D9.1 (A1), J1.0 (PAD), J1.3, J1.5, J1.6, J2.3 (Pin_3), J3.0 (PAD), J3.3, J3.5, J3.6, J4.3 (Pin_3), J5.2 (Pin_2), R22.2, R30.2, RV1.2, SW1.2, SW2.2, SW3.2, U3.23 (VSS), U3.35 (VSS), U3.47 (VSS), U3.8 (VSSA), U4.1 (GND), U6.2 (GND), U6.8 (Rs), U7.1 (A0), U7.2 (A1), U7.3 (A2), U7.4 (GND)
- net VDD: now also J5.1 (Pin_1), RV1.1; no longer C6.1
- net VSen: now also D5.1 (K), JP1.1 (A), R14.1; no longer C5.1, D5.2 (A)
- net at C4.1, M1.2 (-), Q3.1 (S)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: now also RV2.2
- net at C1.1, M1.1 (+), Q1.3 (D)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: now also RV2.1
- net +9V renamed +12V
- net +12V: now also C10.1, D15.2 (A2), D21.1 (K), D22.1 (K), D6.2 (A2), J1.9, J3.9, R29.1, U4.3 (VI); no longer C7.1
- new net: C5.1, JP1.2 (B), R14.2, U3.27 (PB14)
- new net: D18.2 (A2), R25.2, R26.2, SW2.1
- new net: D19.2 (A2), R27.2, R28.2, SW3.1
- new net: C17.2, U3.3 (PC14), Y2.2
- new net: C18.2, U3.4 (PC15), Y2.1
- new net: R20.2, U3.44 (BOOT0)
- new net: C19.2, U3.5 (PF0), Y1.2
- new net: C20.2, U3.6 (PF1), Y1.1
- new net: D17.2 (A2), J4.2 (Pin_2), R24.2
- new net: D11.2 (A2), J2.4 (Pin_4), R18.1
- new net: D16.2 (A2), J4.1 (Pin_1), R23.2
- new net: D12.2 (A2), J2.2 (Pin_2), R17.1
- new net: D10.2 (A2), J2.5 (Pin_5), R19.1
- new net: D14.2 (A2), R15.2, R16.2, SW1.1
- new net +3.3VA: C11.1, C15.1, C16.1, D22.2 (A), D7.1 (K), U3.9 (VDDA), U4.2 (VO)
- new net ADC1_IN13: D20.2 (A2), R29.2, R30.1, U3.26 (PB13)
- new net CAN_H: C22.1, D9.2 (A2), J1.7, J3.7, U6.7 (CANH)
- new net CAN_L: C21.2, D8.1 (A1), J1.2, J3.2, U6.6 (CANL)
- new net CAN_RX_STM: U3.45 (PB8), U6.4 (R)
- new net CAN_TX_STM: U3.46 (PB9), U6.1 (D)
- new net COMP2_OUT: TP4.1, U3.33 (PA12)
- new net COMP4_INM: R21.2, R22.1, U3.20 (PB2)
- new net COMP4_OUT: TP3.1, U3.19 (PB1)
- new net DAC_OUT: TP1.1, U3.14 (PA4)
- new net I2C_SCL: R32.2, U3.38 (PA15), U7.6 (SCL)
- new net I2C_SDA: R31.2, U3.43 (PB7), U7.5 (SDA)
- new net IO_IN1: U3.15 (PA5)
- new net IO_IN2: U3.30 (PA9)
- new net IO_OUT1: U3.39 (PB3), U7.7 (WP)
- new net IO_OUT2: U3.42 (PB6), U6.5 (EN)
- new net IO_OUT3: U3.40 (PB4)
- new net IO_OUT4: U3.41 (PB5)
- new net NRST: R16.1, R19.2, U3.7 (NRST)
- new net OPAMP_OUT: TP2.1, U3.16 (PA6), U3.17 (PA7), U3.18 (PB0)
- new net SWCLK: R17.2, U3.37 (PA14)
- new net SWDIO: R18.2, U3.34 (PA13)
- new net SWO: J2.6 (Pin_6)
- new net TIM1_BKIN: R25.1, U3.25 (PB12)
- new net TIM1_BKIN2: R27.1, U3.32 (PA11)
- new net USART3_RX: R24.1, U3.22 (PB11)
- new net USART3_TX: R23.1, U3.21 (PB10)
- no-connect marks 0 -> 6
Other:
- moved on the sheet: C5, C8, C9, M1, U5
