File: motordriver2.kicad_sch (KiCad schematic)
At the start: 107 parts, among them J1 DE9_Receptacle_MountingHoles, J2 Conn_01x06_Pin, J3 DE9_Receptacle_MountingHoles, J4 Conn_01x03_Pin, J5 Conn_01x02_Pin, M1 Motor_DC, Q1 TPHR9003NL, Q2 TPHR9003NL, Q3 TPHR9003NL, Q4 TPHR9003NL, SW1 SW_Push, SW2 SW_Push, SW3 SW_Push, U1 PLM2105DR, U2 PLM2105DR, U3 STM32F302C8Tx, U4 AMS1117-3.3, U5 AMS1117-3.3, U6 SN65HVD234, U7 24LC256, Y1 X322516MLB4SI, Y2 Q13FC1350000400

Commit message: comp10*10
Parts:
- removed J5: Conn_01x02_Pin, Connector_AMASS:AMASS_XT60IPW-M_1x03_P7.20mm_Horizontal, symbol Connector:Conn_01x02_Pin
- added D12: KT-0805G, Diode_SMD:D_0805_2012Metric, symbol Device:LED
- added D14, D15: ESD3Z5.0C, Diode_SMD:D_SOD-323, symbol Device:D_TVS
- added D7, D8: NCD0805R1, Diode_SMD:D_0805_2012Metric, symbol Device:LED
- added D9: KT-0805Y, Diode_SMD:D_0805_2012Metric, symbol Device:LED
- added H1, H2, H3, H4: MountingHole, MountingHole:MountingHole_2mm, symbol Mechanical:MountingHole
- added J1: Conn_01x02_Pin, Connector_AMASS:AMASS_XT60IPW-M_1x03_P7.20mm_Horizontal, symbol Connector:Conn_01x02_Pin
- added R10, R14, R18, R21: 0805W8F1000T5E, Resistor_SMD:R_0805_2012Metric, symbol Device:R
- added R26, R27: 0805W8F100JT5E, Resistor_SMD:R_0805_2012Metric, symbol Device:R
- added R31, R32: 0402WGF1002TCE, Resistor_SMD:R_0402_1005Metric, symbol Device:R
- added SW1, SW2: TS-1187A-B-A-B, Button_Switch_SMD:SW_Push_1P1T_XKB_TS-1187A, symbol Switch:SW_Push
- added TP2, TP3, TP4, TP5: TestPoint, TestPoint:TestPoint_Loop_D1.80mm_Drill1.0mm_Beaded, symbol Connector:TestPoint
- C21: renamed from C8; footprint (none) -> Capacitor_SMD:C_1206_3216Metric
- C22: renamed from C10; footprint (none) -> Capacitor_SMD:C_1206_3216Metric
- C23: renamed from C9; footprint (none) -> Capacitor_SMD:C_0805_2012Metric
- C24: renamed from C11; footprint (none) -> Capacitor_SMD:C_0805_2012Metric
- C3: renamed from C19; footprint (none) -> Capacitor_SMD:C_0402_1005Metric
- C4: renamed from C20; footprint (none) -> Capacitor_SMD:C_0402_1005Metric
- C7: renamed from C5; footprint (none) -> Capacitor_SMD:C_0805_2012Metric; LCSC C1798 -> C1804
- J2: renamed from J1; value DE9_Receptacle_MountingHoles -> 5788797-1; footprint (none) -> Connector_Dsub:DSUB-9_Female_Horizontal_P2.77x2.84mm_EdgePinOffset7.70mm_Housed_MountingHolesOffset9.12mm
- J3: value DE9_Receptacle_MountingHoles -> 5788797-1; footprint (none) -> Connector_Dsub:DSUB-9_Female_Horizontal_P2.77x2.84mm_EdgePinOffset7.70mm_Housed_MountingHolesOffset9.12mm
- R12: renamed from R11; footprint (none) -> Resistor_SMD:R_0603_1608Metric
- R13: renamed from R12; footprint (none) -> Resistor_SMD:R_0603_1608Metric
- R15: renamed from R9; footprint (none) -> Resistor_SMD:R_0603_1608Metric
- R16: renamed from R10; footprint (none) -> Resistor_SMD:R_0603_1608Metric
- R19: renamed from R7; footprint (none) -> Resistor_SMD:R_0603_1608Metric
- R20: renamed from R8; footprint (none) -> Resistor_SMD:R_0603_1608Metric
- R22: renamed from R21; value R -> 0603WAF3601T5E; footprint (none) -> Resistor_SMD:R_0603_1608Metric; LCSC (none) -> C22980
- R23: renamed from R22; value R -> 0603WAF7501T5E; footprint (none) -> Resistor_SMD:R_0603_1608Metric; LCSC (none) -> C23234
- R24: renamed from R29; value R -> 0603WAF1802T5E; footprint (none) -> Resistor_SMD:R_0603_1608Metric; LCSC (none) -> C25810
- R25: renamed from R30; value R -> 0603WAF2001T5E; footprint (none) -> Resistor_SMD:R_0603_1608Metric; LCSC (none) -> C22975
- R3: renamed from R1; footprint (none) -> Resistor_SMD:R_0603_1608Metric
- R4: renamed from R2; footprint (none) -> Resistor_SMD:R_0603_1608Metric
- R5: renamed from R3; footprint (none) -> Resistor_SMD:R_0603_1608Metric
- R6: renamed from R4; footprint (none) -> Resistor_SMD:R_0603_1608Metric
- R7: renamed from R5; footprint (none) -> Resistor_SMD:R_0603_1608Metric
- R8: renamed from R6; footprint (none) -> Resistor_SMD:R_0603_1608Metric
- R9: renamed from R13; footprint (none) -> 000localproj:R_2728_7142Metric
- SW3: value SW_Push -> TS-1187A-B-A-B; footprint (none) -> Button_Switch_SMD:SW_Push_1P1T_XKB_TS-1187A; LCSC (none) -> C318884
- SW4: renamed from SW2; value SW_Push -> TS-1187A-B-A-B; footprint (none) -> Button_Switch_SMD:SW_Push_1P1T_XKB_TS-1187A; LCSC (none) -> C318884
- SW5: renamed from SW1; value SW_Push -> TS-1187A-B-A-B; footprint (none) -> Button_Switch_SMD:SW_Push_1P1T_XKB_TS-1187A; LCSC (none) -> C318884
- U1: renamed from U6; LCSC (none) -> C99818
- U3: LCSC (none) -> C90795
- U4: renamed from U7; footprint (none) -> Package_SO:SOIC-8_3.9x4.9mm_P1.27mm; LCSC (none) -> C2987263
- Y1: renamed from Y2; footprint (none) -> Crystal:Crystal_SMD_3215-2Pin_3.2x1.5mm
- Y2: renamed from Y1; footprint (none) -> Crystal:Crystal_SMD_3225-4Pin_3.2x2.5mm
- renumbered C23 to C1, C1 to C10, C24 to C11, C15 to C12, C6 to C13, C12 to C14, C13 to C15, C14 to C17, C4 to C18, C7 to C19, C3 to C20, C17 to C5, C18 to C6, C22 to C8, C21 to C9, D5 to D1, D3 to D10, D4 to D11, D20 to D13, D19 to D16, D18 to D17, D14 to D18, D13 to D19, D9 to D2, D6 to D20, D15 to D21, D12 to D22, D11 to D23, D17 to D24, D10 to D25, D21 to D26, D22 to D27, D16 to D28, D8 to D3, D1 to D4, D2 to D5, D7 to D6, J2 to J4, J4 to J5, Q2 to Q1, Q1 to Q2, R14 to R1, R31 to R11, R32 to R17, R20 to R2, R27 to R28, R25 to R29, R16 to R30, R28 to R33, R26 to R34, R15 to R35, R23 to R36, R24 to R37, R17 to R38, R18 to R39, R19 to R40, RV2 to RV1, RV1 to RV2, TP3 to TP1, TP1 to TP6, TP2 to TP7, TP4 to TP8, U1 to U2, U2 to U5, U5 to U6, U4 to U7
Connections:
- net +12V: no longer R24.1
- net +3.3V: now also R31.1, R32.1
- net COMP2_OUT: now also D8.1 (K)
- net COMP4_OUT: now also D7.1 (K)
- net GND: now also D14.1 (A1), D15.1 (A1), J1.1 (Pin_1), R10.2, R14.2, R18.2, R21.2, SW1.2, SW2.2
- net IO_IN1: now also R26.1
- net IO_IN2: now also R27.1
- net IO_OUT3: now also D12.1 (K)
- net IO_OUT4: now also D9.1 (K)
- net VDD: now also R24.1, J1.2 (Pin_2)
- net at C18.1, Q3.1 (S), Q4.3 (D)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: now also M1.1 (+); no longer M1.2 (-)
- net at C10.1, Q1.1 (S), Q2.3 (D)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: now also M1.2 (-); no longer M1.1 (+)
- net at U3.10 (PA0): now also TP2.1
- net at U3.11 (PA1): now also TP3.1
- net at U3.12 (PA2): now also TP4.1
- net at U3.13 (PA3): now also TP5.1
- net CAN_H renamed CAN_P
- net CAN_L renamed CAN_N
- new net: D7.2 (A), R10.1
- new net: D9.2 (A), R18.1
- new net: D15.2 (A2), R27.2, R32.2, SW2.1
- new net: D8.2 (A), R14.1
- new net: D14.2 (A2), R26.2, R31.2, SW1.1
- new net: D12.2 (A), R21.1
- no-connect marks 6 -> 7
Other:
- moved on the sheet: C11, C12, C16, D13, D16, D17, D18, M1, R11, R17, R22, R23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

Commit message: small
Parts:
- removed TP1, TP8: TestPoint, TestPoint:TestPoint_Loop_D1.80mm_Drill1.0mm_Beaded, symbol Connector:TestPoint
- H1, H2, H3, H4: footprint MountingHole:MountingHole_2mm -> MountingHole:MountingHole_3.2mm_M3_Pad
Changed lines of the file:
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@@
     (stroke (width 0) (type default))
   )
-  (wire (pts (xy 93.98 157.48) (xy 110.49 157.48))
-    (stroke (width 0) (type default))
-  )
   (wire (pts (xy 80.01 147.32) (xy 80.01 158.75))
     (stroke (width 0) (type default))
@@
     (stroke (width 0) (type default))
   )
-  (wire (pts (xy 157.48 157.48) (xy 143.51 157.48))
-    (stroke (width 0) (type default))
-  )
   (wire (pts (xy 378.46 134.62) (xy 382.27 134.62))
     (stroke (width 0) (type default))
@@
       (effects (font (size 1.27 1.27)) (justify left))
     )
-    (property "Footprint" "MountingHole:MountingHole_2mm" (at 220.98 259.08 0)
+    (property "Footprint" "MountingHole:MountingHole_3.2mm_M3_Pad" (at 220.98 259.08 0)
       (effects (font (size 1.27 1.27)) hide)
     )
@@
       (effects (font (size 1.27 1.27)) (justify left))
     )
-    (property "Footprint" "MountingHole:MountingHole_2mm" (at 220.98 271.78 0)
+    (property "Footprint" "MountingHole:MountingHole_3.2mm_M3_Pad" (at 220.98 271.78 0)
       (effects (font (size 1.27 1.27)) hide)
     )
@@
       (effects (font (size 1.27 1.27)) (justify left))
     )
-    (property "Footprint" "MountingHole:MountingHole_2mm" (at 220.98 265.43 0)
+    (property "Footprint" "MountingHole:MountingHole_3.2mm_M3_Pad" (at 220.98 265.43 0)
       (effects (font (size 1.27 1.27)) hide)
     )
@@
     )
   )
-  (symbol (lib_id "Connector:TestPoint") (at 93.98 157.48 90) (unit 1)
-    (in_bom yes) (on_board yes) (dnp no) (fields_autoplaced)
-    (property "Reference" "TP1" (at 90.678 152.7007 90)
-      (effects (font (size 1.27 1.27)))
-    )
-    (property "Value" "TestPoint" (at 90.678 155.1249 90)
-      (effects (font (size 1.27 1.27)))
-    )
-    (property "Footprint" "TestPoint:TestPoint_Loop_D1.80mm_Drill1.0mm_Beaded" (at 93.98 152.4 0)
-      (effects (font (size 1.27 1.27)) hide)
-    )
-    (property "Datasheet" "~" (at 93.98 152.4 0)
-      (effects (font (size 1.27 1.27)) hide)
-    )
-    (pin "1")
-    (instances
-      (project "motordriver2"
-        (path "/d34674d6-272e-49ca-bc46-9bcfd7814871"
-          (reference "TP1") (unit 1)
-        )
-      )
-    )
-  )
   (symbol (lib_id "Device:R") (at 205.74 63.5 270) (mirror x) (unit 1)
     (in_bom yes) (on_board yes) (dnp no)
@@
       (effects (font (size 1.27 1.27)) (justify left))
     )
-    (property "Footprint" "MountingHole:MountingHole_2mm" (at 220.98 278.13 0)
+    (property "Footprint" "MountingHole:MountingHole_3.2mm_M3_Pad" (at 220.98 278.13 0)
       (effects (font (size 1.27 1.27)) hide)
     )
@@
         )
       )
-    )
-  )
-  (symbol (lib_id "Connector:TestPoint") (at 157.48 157.48 270) (unit 1)
-    (in_bom yes) (on_board yes) (dnp no) (fields_autoplaced)
-    (property "Reference" "TP8" (at 162.179 156.2679 90)
-      (effects (font (size 1.27 1.27)) (justify left))
-    )
-    (property "Value" "TestPoint" (at 162.179 158.6921 90)
-      (effects (font (size 1.27 1.27)) (justify left))
-    )
-    (property "Footprint" "TestPoint:TestPoint_Loop_D1.80mm_Drill1.0mm_Beaded" (at 157.48 162.56 0)
-      (effects (font (size 1.27 1.27)) hide)
-    )
-    (property "Datasheet" "~" (at 157.48 162.56 0)
-      (effects (font (size 1.27 1.27)) hide)
-    )
-    (pin "1")
-    (instances
-      (project "motordriver2"
-        (path "/d34674d6-272e-49ca-bc46-9bcfd7814871"
-          (reference "TP8") (unit 1)
-        )
-      )

Commit message: mds
Parts:
- J2, J3: value 5788797-1 -> SUB-DRAM-602A-002; LCSC (none) -> C2846087
Changed lines of the file:
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@@
       (effects (font (size 1.27 1.27)) (justify left))
     )
-    (property "Value" "5788797-1" (at 372.872 228.5421 0)
+    (property "Value" "SUB-DRAM-602A-002" (at 372.872 228.5421 0)
       (effects (font (size 1.27 1.27)) (justify left))
     )
@@
       (effects (font (size 1.27 1.27)) hide)
     )
-    (property "LCSC" "" (at 368.3 227.33 0)
+    (property "LCSC" "C2846087 " (at 368.3 227.33 0)
       (effects (font (size 1.27 1.27)) hide)
     )
@@
       (effects (font (size 1.27 1.27)) (justify left))
     )
-    (property "Value" "5788797-1" (at 372.872 190.4421 0)
+    (property "Value" "SUB-DRAM-602A-002" (at 372.872 190.4421 0)
       (effects (font (size 1.27 1.27)) (justify left))
     )
@@
       (effects (font (size 1.27 1.27)) hide)
     )
-    (property "LCSC" "" (at 368.3 189.23 0)
+    (property "LCSC" "C2846087 " (at 368.3 189.23 0)
       (effects (font (size 1.27 1.27)) hide)
     )

Commit message: change
Parts:
- removed C12: CL05B103KB5NNNC, Capacitor_SMD:C_0402_1005Metric, symbol Device:C
- removed C13, C17: CL05B104KO5NNNC, Capacitor_SMD:C_0402_1005Metric, symbol Device:C
- removed C16, C20: CL10A105KB8NNNC, Capacitor_SMD:C_0603_1608Metric, symbol Device:C
- removed C18: CL21B224KBFNNNE, Capacitor_SMD:C_0805_2012Metric, symbol Device:C
- removed C19: CL10A475KO8NNNC, Capacitor_SMD:C_0603_1608Metric, symbol Device:C
- removed C22: CL31B105KBHNNNE, Capacitor_SMD:C_1206_3216Metric, symbol Device:C
- removed C24: CL21A226MAQNNNE, Capacitor_SMD:C_0805_2012Metric, symbol Device:C
- removed C5, C8: 0402CG150J500NT, Capacitor_SMD:C_0402_1005Metric, symbol Device:C
- removed C7: CL21C200JBANNNC, Capacitor_SMD:C_0805_2012Metric, symbol Device:C
- removed D1: ESD9X3.3ST5G, Diode_SMD:D_SOD-923, symbol Device:D
- removed D10, D11, D27, D4, D5, D6: SS34, Diode_SMD:D_MELF, symbol Device:D
- removed D12: KT-0805G, Diode_SMD:D_0805_2012Metric, symbol Device:LED
- removed D13, D20, D21: ES0402V014BT, Diode_SMD:D_0402_1005Metric, symbol Device:D_TVS
- removed D14, D15, D16, D17, D18, D19, D2, D22, D23, D24, D25, D28, D3: ESD3Z5.0C, Diode_SMD:D_SOD-323, symbol Device:D_TVS
- removed D7, D8: NCD0805R1, Diode_SMD:D_0805_2012Metric, symbol Device:LED
- removed D9: KT-0805Y, Diode_SMD:D_0805_2012Metric, symbol Device:LED
- removed J3: SUB-DRAM-602A-002, Connector_Dsub:DSUB-9_Female_Horizontal_P2.77x2.84mm_EdgePinOffset7.70mm_Housed_MountingHolesOffset9.12mm, symbol Connector:DE9_Receptacle_MountingHoles
- removed J4: Conn_01x06_Pin, Connector_PinSocket_2.54mm:PinSocket_1x06_P2.54mm_Vertical, symbol Connector:Conn_01x06_Pin
- removed J5: Conn_01x03_Pin, Connector_PinSocket_2.54mm:PinSocket_1x03_P2.54mm_Vertical, symbol Connector:Conn_01x03_Pin
- removed JP1: Jumper_2_Open, Jumper:SolderJumper-2_P1.3mm_Open_Pad1.0x1.5mm, symbol Jumper:Jumper_2_Open
- removed R10, R14, R21: 0805W8F1000T5E, Resistor_SMD:R_0805_2012Metric, symbol Device:R
- removed R11, R17: 0805W8F3301T5E, Resistor_SMD:R_0805_2012Metric, symbol Device:R
- removed R22: 0603WAF3601T5E, Resistor_SMD:R_0603_1608Metric, symbol Device:R
- removed R23: 0603WAF7501T5E, Resistor_SMD:R_0603_1608Metric, symbol Device:R
- removed R27, R28, R29, R30, R36, R37, R38, R39, R40: 0805W8F100JT5E, Resistor_SMD:R_0805_2012Metric, symbol Device:R
- removed R32, R33, R34, R35: 0402WGF1002TCE, Resistor_SMD:R_0402_1005Metric, symbol Device:R
- removed R9: HoXLR2728D-4W-7mR-1%, 000localproj:R_2728_7142Metric, symbol Device:R
- removed SW2, SW4, SW5: TS-1187A-B-A-B, Button_Switch_SMD:SW_Push_1P1T_XKB_TS-1187A, symbol Switch:SW_Push
- removed TP2, TP3, TP4, TP5, TP6, TP7: TestPoint, TestPoint:TestPoint_Loop_D1.80mm_Drill1.0mm_Beaded, symbol Connector:TestPoint
- removed U1: SN65HVD234, Package_SO:SOIC-8_3.9x4.9mm_P1.27mm, symbol Interface_CAN_LIN:SN65HVD234
- removed U2, U5: PLM2105DR, SOIC8_D_TEX, symbol 0000locallib:PLM2105DR
- removed U3: STM32F302C8Tx, Package_QFP:LQFP-48_7x7mm_P0.5mm, symbol MCU_ST_STM32F3:STM32F302C8Tx
- removed U4: 24LC256, Package_SO:SOIC-8_3.9x4.9mm_P1.27mm, symbol Memory_EEPROM:24LC256
- removed U6, U7: AMS1117-3.3, Package_TO_SOT_SMD:SOT-223-3_TabPin2, symbol Regulator_Linear:AMS1117-3.3
- removed Y1: Q13FC1350000400, Crystal:Crystal_SMD_3215-2Pin_3.2x1.5mm, symbol Device:Crystal
- removed Y2: X322516MLB4SI, Crystal:Crystal_SMD_3225-4Pin_3.2x2.5mm, symbol Device:Crystal
- added C10: CL10B104MB8NNNC, Capacitor_SMD:C_0603_1608Metric, symbol Device:C
- added D7, D8: SK6812MINI, LED_SMD:LED_SK6812MINI_PLCC4_3.5x3.5mm_P1.75mm, symbol LED:SK6812MINI
- added J3: ICSP, Connector_PinSocket_2.54mm:PinSocket_1x08_P2.54mm_Vertical, symbol Connector:Conn_01x08_Pin
- added J4: FAN, Connector_PinSocket_2.54mm:PinSocket_1x03_P2.54mm_Vertical, symbol Connector:Conn_01x03_Pin
- added Q5: AO3400A, Package_TO_SOT_SMD:SOT-23, symbol Transistor_FET:AO3400A
- added R12: RC0603JR-0751KL, Resistor_SMD:R_0603_1608Metric, symbol Device:R
- added R13: RC0603JR-071K8L, Resistor_SMD:R_0603_1608Metric, symbol Device:R
- added R5: RC0603JR-1310KL, Resistor_SMD:R_0603_1608Metric, symbol Device:R
- added R6: 0.008, Resistor_SMD:R_2512_6332Metric_Pad1.40x3.35mm_HandSolder, symbol Device:R
- added R7: RC0603JR-10470RL, Resistor_SMD:R_0603_1608Metric, symbol Device:R
- added RV1, RV2: SDV1608H260C050YPTF, Resistor_SMD:R_0603_1608Metric, symbol Device:Varistor
- added RV4, RV7: AVR-M1005C080MTADB, Resistor_SMD:R_0402_1005Metric, symbol Device:Varistor
- added U1: LM358, Package_SO:SOIC-8_3.9x4.9mm_P1.27mm, symbol Amplifier_Operational:LM358
- added U2, U7: MCP14700T-E/SN, Package_SO:SOIC-8_3.9x4.9mm_P1.27mm, symbol 0000locallib:MCP14700T-E_SN
- added U3: PIC16F1829-ISS, Package_SO:SSOP-20_5.3x7.2mm_P0.65mm, symbol MCU_Microchip_PIC16:PIC16F1829-ISS
- added U5: TMP1075DGK, Package_SO:VSSOP-8_3.0x3.0mm_P0.65mm, symbol Sensor_Temperature:TMP1075DGK
- added U6: L78M05ABDT-TR, Package_TO_SOT_SMD:TO-252-2, symbol Regulator_Linear:LT1129-3.3_SOT223
- C1: value CL05B104KO5NNNC -> CL10X106MO8NRNC; footprint Capacitor_SMD:C_0402_1005Metric -> Capacitor_SMD:C_0603_1608Metric; LCSC C1525 -> C19702
- C11: value CL10A475KO8NNNC -> CL10A105KA8NNNL; LCSC C19666 -> C15849
- C12: renamed from C21; value CL31B105KBHNNNE -> CL10A105KA8NNNL; footprint Capacitor_SMD:C_1206_3216Metric -> Capacitor_SMD:C_0603_1608Metric_Pad1.08x0.95mm_HandSolder
- C13: renamed from C23; value CL21A226MAQNNNE -> GCM188N8EA226ME08J; footprint Capacitor_SMD:C_0805_2012Metric -> Capacitor_SMD:C_0603_1608Metric_Pad1.08x0.95mm_HandSolder
- C14: value CL05B104KO5NNNC -> CL10B104MB8NNNC; footprint Capacitor_SMD:C_0402_1005Metric -> Capacitor_SMD:C_0603_1608Metric; LCSC C1525 -> C14663
- C15: value CL05B104KO5NNNC -> CL21B224KBFNNNE; footprint Capacitor_SMD:C_0402_1005Metric -> Capacitor_SMD:C_0805_2012Metric; LCSC C1525 -> C5378
- C2: value CL10A105KB8NNNC -> CL10A105KA8NNNL
- C3: value CL05C100JB5NNNC -> CL10B104MB8NNNC; footprint Capacitor_SMD:C_0402_1005Metric -> Capacitor_SMD:C_0603_1608Metric; LCSC C32949 -> C14663
- C4: value CL05C100JB5NNNC -> CL10X106MO8NRNC; footprint Capacitor_SMD:C_0402_1005Metric -> Capacitor_SMD:C_0603_1608Metric; LCSC C32949 -> C19702
- C6, C9: value 0402CG150J500NT -> CL10B104MB8NNNC; footprint Capacitor_SMD:C_0402_1005Metric -> Capacitor_SMD:C_0603_1608Metric; LCSC C1548 -> C14663
- D9: renamed from D26; value SS34 -> RS1M; footprint Diode_SMD:D_MELF -> Diode_SMD:D_SMA_Handsoldering
- J2: value SUB-DRAM-602A-002 -> DMR-09PGG
- Q1, Q2, Q3, Q4: value TPHR9003NL -> TPN1R603PLL1Q; footprint Package_SON:VSONP-8-1EP_5x6_P1.27mm -> 000localproj:TSON Advance_TOS; LCSC C129784 -> C516183
- R1: value 0805W8F100JT5E -> RC0603JR-1310KL; footprint Resistor_SMD:R_0805_2012Metric -> Resistor_SMD:R_0603_1608Metric; LCSC C17415 -> C25744
- R10: renamed from R7; value 0603WAF1002T5E -> RC0603JR-1310KL
- R11: renamed from R8; value 0603WAF1002T5E -> RC0603JR-1310KL
- R14: renamed from R12; value 0603WAF1002T5E -> RC0603JR-1310KL
- R15: renamed from R13; value 0603WAF1002T5E -> RC0603JR-1310KL
- R16: renamed from R15; value 0603WAF470JT5E -> RC0603JR-10470RL
- R17: renamed from R16; value 0603WAF470JT5E -> RC0603JR-10470RL
- R18: value 0805W8F1000T5E -> 0.008; footprint Resistor_SMD:R_0805_2012Metric -> Resistor_SMD:R_2512_6332Metric_Pad1.40x3.35mm_HandSolder; LCSC C17408 -> (none)
- R19, R20: value 0603WAF470JT5E -> 0.008; footprint Resistor_SMD:R_0603_1608Metric -> Resistor_SMD:R_2512_6332Metric_Pad1.40x3.35mm_HandSolder; LCSC C23182 -> (none)
- R2: value 0402WGF1002TCE -> RC0603JR-1310KL; footprint Resistor_SMD:R_0402_1005Metric -> Resistor_SMD:R_0603_1608Metric
- R22: renamed from R31; value 0402WGF1002TCE -> RC0603JR-1310KL; footprint Resistor_SMD:R_0402_1005Metric -> Resistor_SMD:R_0603_1608Metric
- R24: value 0603WAF1802T5E -> RC0603JR-10100RL; LCSC C25810 -> C17415
- R25: value 0603WAF2001T5E -> RC0603JR-10100RL; LCSC C22975 -> C17415
- R26: value 0805W8F100JT5E -> RC0603JR-10100RL; footprint Resistor_SMD:R_0805_2012Metric -> Resistor_SMD:R_0603_1608Metric
- R3: value 0603WAF470JT5E -> RC0603JR-079K1L; LCSC C23182 -> C23260
- R4: value 0603WAF470JT5E -> RC0603JR-0775KL; LCSC C23182 -> C23242
- R8: renamed from R5; value 0603WAF470JT5E -> RC0603JR-10470RL
- R9: renamed from R6; value 0603WAF470JT5E -> RC0603JR-10470RL
- renumbered C10 to C5, RV1 to RV3, RV2 to RV6
Connections:
- net GATEHA: now also U2.2 (PWMHI), U3.5 (RC5)
- net GATEHB: now also U3.15 (RC1), U7.2 (PWMHI)
- net GATELA: now also U2.3 (PWMLO), U3.6 (RC4)
- net GATELB: now also U3.16 (RC0), U7.3 (PWMLO)
- net GND: now also C3.2, C4.2, C6.2, C9.2, R19.2, R20.2, R3.1, C10.2, D7.2 (VSS), D8.2 (VSS), J3.3 (Pin_3), Q5.2 (S), R13.1, R6.2, RV1.2, RV2.1, RV4.2, RV7.2, U1.4 (V-), U2.4 (GND), U3.20 (VSS), U5.4 (GND), U5.5 (A2), U5.6 (A1), U5.7 (A0), U6.2 (GND), U7.4 (GND); no longer C15.2, C3.1, C4.1, C6.1, C9.1, J2.3, R25.2
- net VDD: now also C12.1, D9.1 (K), J4.2 (Pin_2), U6.1 (VI); no longer R24.1
- net VSen: now also R18.1, R19.1, R20.1, R6.1, RV2.2, U1.3 (+); no longer R1.1
- net at R16.1: now also U7.8 (HIGHDR); no longer R19.2
- net at M1.1 (+), Q3.1 (S), Q4.3 (D)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: now also C15.1, U7.1 (PHASE)
- net SDA: now reaches R1.2
- net SDA: now also U3.13 (RB4), U5.1 (SDA)
- net IN1: now reaches R22.2, SW1.1
- net IN1: now also C10.1, RV4.1, U3.17 (RA2); no longer R26.2
- net IN2: now reaches R4.1
- net IN2: now also R3.2, U1.2 (-)
- net voltage_motor: now reaches C5.1, M1.2 (-), Q1.1 (S), Q2.3 (D), R10.1, RV3.1
- net voltage_motor: now also R12.1, RV1.1, U2.1 (PHASE)
- net at C5.2: now also U2.7 (BOOT)
- net MCLR*: now reaches SW3.1
- net MCLR*: now also C14.1, R24.1, R5.2, RV7.1, U3.4 (RA3/MCLR/VPP)
- net SCL: now reaches R2.2
- net SCL: now also U3.11 (RB6), U5.2 (SCL)
- net at R17.1: now also U7.5 (LOWDR); no longer R20.2
- net at R9.1: now also U2.5 (LOWDR); no longer R4.2
- net at R8.1: now also U2.8 (HIGHDR); no longer R3.2
- removed net +12V: C12.1, C2.1, D9.1 (K), J2.9
- net +3.3V renamed +5V
- net +5V: now also C2.1, C3.1, C4.1, C6.1, C9.1, R1.1, D7.4 (VDD), D8.4 (VDD), J3.2 (Pin_2), R5.1, U1.8 (V+), U2.6 (VCC), U3.1 (VDD), U5.8 (V+), U6.3 (VO), U7.6 (VCC); no longer C14.1, C15.1
- net ADC1_IN13: no longer names the net of R24.2
- net ADC1_IN13: now also J3.1 (Pin_1); no longer R25.1
- net CAN_N renamed PIC_UART_TX
- net PIC_UART_TX: now also U3.10 (RB7); no longer C9.2
- net CAN_P: no longer names the net of J2.7
- net IO_IN1 renamed PGC
- net PGC: now also U3.18 (RA1/ICSPCLK)
- new net: J3.4 (Pin_4), R25.2
- new net: J3.5 (Pin_5), R26.2
- new net: D7.1 (DOUT), D8.3 (DIN)
- new net: R12.2, R13.2, U1.5 (+)
- new net: Q5.1 (G), R7.1
- new net: C15.2, U7.7 (BOOT)
- new net: J4.3 (Pin_3), Q5.3 (D)
- new net FAN: R7.2, U3.2 (RA5)
- new net INT: U3.3 (RA4), U5.3 (ALERT)
- new net ISenseIN: R4.2, U1.1, U3.14 (RC2), U3.9 (RC7)
- new net LED: D7.3 (DIN), U3.7 (RC3)
- new net PGD: R25.1, U3.19 (RA0/ICSPDAT)
- new net PIC_UART_RX: J2.3, U3.12 (RB5)
- new net VSenseIN: U1.6 (-), U1.7, U3.8 (RC6)
- no-connect marks 7 -> 10
Other:
- moved on the sheet: C12, C13, C2, D9, H1, H2, H3, H4, J2

Commit message: add production
Parts:
- removed C11: CL10A105KA8NNNL, Capacitor_SMD:C_0603_1608Metric, symbol Device:C
- removed C15: CL21B224KBFNNNE, Capacitor_SMD:C_0805_2012Metric, symbol Device:C
- removed D7, D8: SK6812MINI, LED_SMD:LED_SK6812MINI_PLCC4_3.5x3.5mm_P1.75mm, symbol LED:SK6812MINI
- removed R20: 0.008, Resistor_SMD:R_2512_6332Metric_Pad1.40x3.35mm_HandSolder, symbol Device:R
- removed U2, U7: MCP14700T-E/SN, Package_SO:SOIC-8_3.9x4.9mm_P1.27mm, symbol 0000locallib:MCP14700T-E_SN
- removed U3: PIC16F1829-ISS, Package_SO:SSOP-20_5.3x7.2mm_P0.65mm, symbol MCU_Microchip_PIC16:PIC16F1829-ISS
- added C7: CL10A105KA8NNNL, Capacitor_SMD:C_0603_1608Metric, symbol Device:C
- added C8: CL21B224KBFNNNE, Capacitor_SMD:C_0805_2012Metric, symbol Device:C
- added D1: LED, LED_SMD:LED_0603_1608Metric_Pad1.05x0.95mm_HandSolder, symbol Device:LED
- added J5: Conn_01x02_Socket, Connector_PinSocket_2.54mm:PinSocket_1x02_P2.54mm_Vertical, symbol Connector:Conn_01x02_Socket
- added J6: Encoder, Connector_PinSocket_2.54mm:PinSocket_1x03_P2.54mm_Vertical, symbol Connector:Conn_01x03_Pin
- added JP1: SolderJumper_2_Bridged, Jumper:SolderJumper-2_P1.3mm_Bridged_RoundedPad1.0x1.5mm, symbol Jumper:SolderJumper_2_Bridged
- added R21: RC0603JR-10100RL, Resistor_SMD:R_0603_1608Metric, symbol Device:R
- added U2, U4: PLM2105DR, 000localproj:SOIC8_D_TEX, symbol 0000locallib:PLM2105DR
- added U7: PIC16F18344-SS, Package_SO:SSOP-20_5.3x7.2mm_P0.65mm, symbol MCU_Microchip_PIC16:PIC16F18344-SS
- R13: value RC0603JR-071K8L -> RC0603JR-1310KL; LCSC C4177 -> C25744
- R18: value 0.008 -> RC0603JR-0751KL; footprint Resistor_SMD:R_2512_6332Metric_Pad1.40x3.35mm_HandSolder -> Resistor_SMD:R_0603_1608Metric; LCSC (none) -> C23196
- R19: value 0.008 -> RC0603JR-1310KL; footprint Resistor_SMD:R_2512_6332Metric_Pad1.40x3.35mm_HandSolder -> Resistor_SMD:R_0603_1608Metric; LCSC (none) -> C25744
- R3: value RC0603JR-079K1L -> RC0603JR-071KL; LCSC C23260 -> (none)
- R4: value RC0603JR-0775KL -> RC0603JR-1310KL; LCSC C23242 -> C25744
- R6: value 0.008 -> PMR100HZPFU5L00; footprint Resistor_SMD:R_2512_6332Metric_Pad1.40x3.35mm_HandSolder -> Resistor_SMD:R_2512_6332Metric
Connections:
- net PGC is gone; now on net ISenseIN: R26.1
- net +5V: now also U7.1 (VDD); no longer C2.1
- net FAN: now also U7.8 (RC6)
- net GATEHA: now also U4.2 (INH), U7.17 (RA2)
- net GATEHB: now also U2.2 (INH), U7.15 (RC1)
- net GATELA: now also U4.3 (INL), U7.16 (RC0)
- net GATELB: now also U2.3 (INL), U7.14 (RC2)
- net GND: now also R19.1, R3.2, R4.2, C7.2, D1.1 (K), J5.2 (Pin_2), J6.3 (Pin_3), U2.4 (GND), U4.4 (GND), U7.20 (VSS); no longer R18.2, R19.2, R3.1
- net IN1: now also U7.9 (RC7)
- net IN2: now also R18.2, R3.1; no longer R3.2, R4.1
- net INT: now also U7.5 (RC5)
- net ISenseIN: now also R13.2, R18.1, U7.18 (RA1/ICSPCLK); no longer R4.2
- net LED: now also R21.2, U7.7 (RC3)
- net MCLR*: now also U7.4 (RA3/~{MCLR}/VPP)
- net PGD: now also R19.2, U7.19 (RA0/ICSPDAT)
- net PIC_UART_RX: now also U7.12 (RB5)
- net PIC_UART_TX: now also U7.10 (RB7)
- net SCL: now also U7.11 (RB6)
- net SDA: now also U7.13 (RB4)
- net VDD: now also JP1.2 (B); no longer J4.2 (Pin_2)
- net VSen: no longer R18.1, R19.1
- net VSenseIN: now also U7.6 (RC4)
- net voltage_motor: now also U4.6 (SH)
- net at M1.1 (+), Q3.1 (S), Q4.3 (D)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: now also C8.1, U2.6 (SH)
- net at C5.2: now also U4.8 (BST)
- net at R9.1: now also U4.5 (GL)
- net at R12.2, U1.5 (+): now also R4.1; no longer R13.2
- net at R17.1: now also U2.5 (GL)
- net at R8.1: now also U4.7 (GH)
- net at R16.1: now also U2.7 (GH)
- new net: D1.2 (A), R21.1
- new net: C8.2, U2.8 (BST)
- new net +12V: C2.1, C7.1, J4.2 (Pin_2), J5.1 (Pin_1), JP1.1 (A), U2.1 (GVDD), U4.1 (GVDD)
- new net ENC1: J6.1 (Pin_1), U7.3 (RA4)
- new net ENC2: J6.2 (Pin_2), U7.2 (RA5)
- no-connect marks 10 -> 9
Other:
- moved on the sheet: C2, R5
